File: receiver/RC_Car_receiver.kicad_sch (KiCad schematic)
At the start: 74 parts, among them M1 STEERING_MOTOR, M2 PRIMARY_MOTOR, Q1 2SC3192-O_ECB, Q10 2SC468-C_ECB, Q11 2SA733-P_ECB, Q12 H8550-C_ECB, Q13 H8550-C_ECB, Q14 H8050-C_ECB, Q15 H8050-C_ECB, Q2 2SC945-P_ECB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

Commit message: add scope photos
Other:
- added sheet Waveforms (waveforms.kicad_sch)
Changed lines of the file:
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@@
+    )
+  )
+  (sheet (at 234.315 152.4) (size 12.7 12.065) (fields_autoplaced)
+    (stroke (width 0.1524) (type solid))
+    (fill (color 0 0 0 0.0000))
+    (property "Sheetname" "Waveforms" (at 234.315 151.6884 0)
+      (effects (font (size 1.27 1.27) bold) (justify left bottom))
+    )
+    (property "Sheetfile" "waveforms.kicad_sch" (at 234.315 165.0496 0)
+      (effects (font (size 1.27 1.27)) (justify left top))
+    )
+    (instances
+      (project "RC_Car_receiver"
+        (path "/e63e39d7-6ac0-4ffd-8aa3-1841a4541b55" (page "2"))
+      )
     )
   )

Commit message: add scope waveform photos
Parts:
- gave numbers to parts that had none: 1
Changed lines of the file:
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@@
   (symbol (lib_id "Device:Antenna") (at 52.705 22.86 0) (unit 1)
     (in_bom yes) (on_board yes) (dnp no) (fields_autoplaced)
-    (property "Reference" "AE?" (at 54.737 22.5865 0)
-      (effects (font (size 1.27 1.27)) (justify left))
-    )
-    (property "Value" "Antenna" (at 54.737 25.3616 0)
+    (property "Reference" "AE1" (at 54.737 22.2829 0)
+      (effects (font (size 1.27 1.27)) (justify left))
+    )
+    (property "Value" "Antenna" (at 54.737 24.7071 0)
       (effects (font (size 1.27 1.27)) (justify left))
     )
@@
       (project "RC_Car_receiver"
         (path "/e63e39d7-6ac0-4ffd-8aa3-1841a4541b55"
-          (reference "AE?") (unit 1)
+          (reference "AE1") (unit 1)
         )
       )
@@
     )
   )
-  (sheet (at 234.315 152.4) (size 12.7 12.065) (fields_autoplaced)
+  (sheet (at 240.665 156.21) (size 12.7 12.065) (fields_autoplaced)
     (stroke (width 0.1524) (type solid))
     (fill (color 0 0 0 0.0000))
-    (property "Sheetname" "Waveforms" (at 234.315 151.6884 0)
+    (property "Sheetname" "Waveforms" (at 240.665 155.4984 0)
       (effects (font (size 1.27 1.27) bold) (justify left bottom))
     )
-    (property "Sheetfile" "waveforms.kicad_sch" (at 234.315 165.0496 0)
+    (property "Sheetfile" "waveforms.kicad_sch" (at 240.665 168.8596 0)
       (effects (font (size 1.27 1.27)) (justify left top))
     )
