File: receiver/waveforms.kicad_sch (KiCad schematic)
At the start: 0 parts

Commit message: add scope waveform photos
Other:
- note added: "All signals referenced to GND (not GNDA)"
- note added: "TP1 Detector Out AC Coupled"
- note added: "TP1 Detector Out DC Coupled"
- note added: "TP2 AF Amp Out"
- note added: "TP3 Logic Converter Out"
- note added: "Transmitter OFF"
- note added: "Transmitter ON"
- title: (none) -> Marcraft SE-1030 RC Car (Confluent)
Changed lines of the file:
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@@
 (kicad_sch (version 20230121) (generator eeschema)
-  (paper "A4")
-  (image (at 46.355 126.365)
+  (paper "A")
+  (title_block
+    (title "Marcraft SE-1030 RC Car (Confluent)")
+    (date "2023-07-22")
+  )
+  (image (at 49.53 130.81)
     (data
       iVBORw0KGgoAAAANSUhEUgAAAyAAAAHgCAIAAADSZZ6iAAAAA3NCSVQICAjb4U/gAAAgAElEQVR4
@@
     )
   )
-  (image (at 46.99 34.29)
+  (image (at 49.53 45.085)
     (data
       iVBORw0KGgoAAAANSUhEUgAAAyAAAAHgCAIAAADSZZ6iAAAAA3NCSVQICAjb4U/gAAAgAElEQVR4
@@
     )
   )
-  (image (at 44.45 78.74)
+  (image (at 49.53 88.265)
     (data
       iVBORw0KGgoAAAANSUhEUgAAAyAAAAHgCAIAAADSZZ6iAAAAA3NCSVQICAjb4U/gAAAgAElEQVR4
@@
     )
   )
-  (image (at 127 128.905)
+  (image (at 132.08 130.81)
     (data
       iVBORw0KGgoAAAANSUhEUgAAAyAAAAHgCAIAAADSZZ6iAAAAA3NCSVQICAjb4U/gAAAgAElEQVR4
@@
     )
   )
-  (image (at 125.095 32.385)
+  (image (at 132.08 45.085)
     (data
       iVBORw0KGgoAAAANSUhEUgAAAyAAAAHgCAIAAADSZZ6iAAAAA3NCSVQICAjb4U/gAAAgAElEQVR4
@@
     )
   )
-  (image (at 126.365 81.28)
+  (image (at 132.08 88.265)
     (data
       iVBORw0KGgoAAAANSUhEUgAAAyAAAAHgCAIAAADSZZ6iAAAAA3NCSVQICAjb4U/gAAAgAElEQVR4
@@
     )
   )
-  (image (at 50.165 172.72)
+  (image (at 49.53 173.99)
     (data
       iVBORw0KGgoAAAANSUhEUgAAAyAAAAHgCAIAAADSZZ6iAAAAA3NCSVQICAjb4U/gAAAgAElEQVR4
@@
     )
   )
-  (image (at 126.365 173.99)
+  (image (at 132.08 173.99)
     (data
       iVBORw0KGgoAAAANSUhEUgAAAyAAAAHgCAIAAADSZZ6iAAAAA3NCSVQICAjb4U/gAAAgAElEQVR4
@@
     )
   )
+  (text "TP1 Detector Out\nAC Coupled" (at 41.275 103.505 0)
+    (effects (font (size 1.27 1.27) (thickness 0.254) bold (color 255 255 255 1)) (justify left bottom))
+  )
+  (text "TP1 Detector Out\nDC Coupled" (at 40.64 59.69 0)
+    (effects (font (size 1.27 1.27) (thickness 0.254) bold (color 255 255 255 1)) (justify left bottom))
+  )
+  (text "TP2 AF Amp Out" (at 40.64 146.05 0)
+    (effects (font (size 1.27 1.27) (thickness 0.254) bold (color 255 255 255 1)) (justify left bottom))
+  )
+  (text "Transmitter OFF" (at 38.735 20.955 0)
+    (effects (font (size 1.905 1.905) (thickness 0.254) bold) (justify left bottom))
+  )
+  (text "TP3 Logic Converter Out" (at 121.285 189.23 0)
+    (effects (font (size 1.27 1.27) (thickness 0.254) bold (color 255 255 255 1)) (justify left bottom))
+  )
+  (text "TP3 Logic Converter Out" (at 36.83 189.23 0)
+    (effects (font (size 1.27 1.27) (thickness 0.254) bold (color 255 255 255 1)) (justify left bottom))
+  )
+  (text "TP1 Detector Out\nAC Coupled" (at 124.46 104.14 0)
+    (effects (font (size 1.27 1.27) (thickness 0.254) bold (color 255 255 255 1)) (justify left bottom))
+  )
+  (text "Transmitter ON" (at 120.015 20.955 0)
+    (effects (font (size 1.905 1.905) (thickness 0.254) bold) (justify left bottom))
+  )
+  (text "TP1 Detector Out\nDC Coupled" (at 123.825 60.325 0)
+    (effects (font (size 1.27 1.27) (thickness 0.254) bold (color 255 255 255 1)) (justify left bottom))
+  )
+  (text "All signals referenced to GND\n(not GNDA)" (at 194.945 170.18 0)
+    (effects (font (size 1.905 1.905) (thickness 0.254) bold) (justify left bottom))
+  )
+  (text "TP2 AF Amp Out" (at 125.095 146.05 0)
+    (effects (font (size 1.27 1.27) (thickness 0.254) bold (color 255 255 255 1)) (justify left bottom))
+  )
 )
